Commit message: Add base_link definition to sensors.xacro for standalone TF verification

File: m8_sensor_kit_description/urdf/sensors.xacro (robot description, xacro)
@@ -1,4 +1,5 @@
 <?xml version="1.0"?>
 <robot name="vehicle" xmlns:xacro="http://ros.org/wiki/xacro">
+  <link name="base_link"/>
   <xacro:arg name="config_dir" default="$(find m8_sensor_kit_description)/config"/>
   <xacro:property name="calibration" value="${xacro.load_yaml('$(arg config_dir)/sensors_calibration.yaml')}"/>
